File: julio_cool_clock/julio_cool_clock.kicad_sch (KiCad schematic)
At the start: 60 parts, among them J1 PJ-102AH, J2 Conn_02x03_Odd_Even, J3 Conn_01x06, Q1 NPN_2N3904_SOT23, SW1 Omron_B3F_SPST, SW2 Omron_B3F_SPST, SW3 Omron_B3F_SPST, SW4 Omron_B3F_SPST, U1 ATmega328-PU, U2 MAX7219, U3 DS1307_DIP-8, U4 L7805, Y1 Crystal_16MHz, Y2 Crystal_32768Hz

Commit message: Final Gerber
Git commit for final Gerber Out. I forgot to upload the Google Form for the initial Gerber but everything from the first one is in the previous Git commit.
Parts:
- added TP15, TP16, TP17, TP18, TP19, TP20: TestPoint, footprints:TestPoint_THTPad_D2.0mm_Drill1.0mm, symbol HPS:TestPoint
- renumbered TP13 to TP14
Connections:
- net DIS_CLK: now also TP18.1
- net DIS_DATA: now also TP17.1
- net DIS_LOAD: now also TP16.1
- net LED_SCK: now also TP15.1
- net SCL: now also TP19.1
- net SDA: now also TP20.1

Commit message: Gerber Out Revisions 1
Parts:
- removed TP2, TP3, TP4, TP6, TP7, TP9: TestPoint, footprints:TestPoint_THTPad_D2.0mm_Drill1.0mm, symbol HPS:TestPoint
Connections:
- net GND: now also U1.22 (GND); no longer TP11.1
- net at DS1.15 (LED(+)), R7.1: now also TP11.1
- net LCD_1 renamed RS
- net LCD_2 renamed E
- net LCD_3 renamed D4
- net LCD_4 renamed D5
- net LCD_5 renamed D6
- net LCD_6 renamed D7
- no-connect marks 10 -> 11
Other:
- moved on the sheet: R7, TP11
