File: julio_cool_clock/_autosave-julio_cool_clock.kicad_pcb (KiCad board)
At the start: 2 copper layers, 140 x 90 mm, 60 parts, among them J1 VAL**, J2 Conn_02x03_Odd_Even, J3 Conn_01x06, Q1 NPN_2N3904_SOT23, SW1 Omron_B3F_SPST, SW2 Omron_B3F_SPST, SW3 Omron_B3F_SPST, SW4 Omron_B3F_SPST, U1 ATmega328-PU, U2 MAX7219, U3 DS1307_DIP-8, U4 L7805, Y1 Crystal_16MHz, Y2 Crystal_32768Hz

Commit message: Final Gerber
Git commit for final Gerber Out. I forgot to upload the Google Form for the initial Gerber but everything from the first one is in the previous Git commit.
Parts:
- added TP15: TestPoint, footprints:TestPoint_THTPad_D2.0mm_Drill1.0mm, F.Cu at (121.2, 81.0)
- added TP16: TestPoint, footprints:TestPoint_THTPad_D2.0mm_Drill1.0mm, F.Cu at (98.0, 140.0)
- added TP17: TestPoint, footprints:TestPoint_THTPad_D2.0mm_Drill1.0mm, F.Cu at (103.0, 140.0)
- added TP18: TestPoint, footprints:TestPoint_THTPad_D2.0mm_Drill1.0mm, F.Cu at (108.0, 140.0)
- added TP19: TestPoint, footprints:TestPoint_THTPad_D2.0mm_Drill1.0mm, F.Cu at (113.8, 87.5)
- added TP20: TestPoint, footprints:TestPoint_THTPad_D2.0mm_Drill1.0mm, F.Cu at (107.2, 97.2)
- J1: value VAL** -> PJ-102AH
- moved J1 5.12 mm to (202.6, 134.7), turned to 180 degrees
Routing:
- net Net-(C7-Pad1): track 22.6 -> 59.8 mm
- net SCL: track 52.0 -> 74.5 mm, vias 2 -> 5
- net SDA: track 45.1 -> 54.0 mm
- net DIS_DATA: track 140.2 -> 147.9 mm
- net LED_SCK: track 55.0 -> 62.5 mm
- net DIS_CLK: track 99.0 -> 104.2 mm
- net DIS_LOAD: track 117.6 -> 121.8 mm
