File: julio_cool_clock/julio_cool_clock.kicad_pcb (KiCad board)
At the start: 2 copper layers, 140 x 90 mm, 60 parts, among them J1 VAL**, J2 Conn_02x03_Odd_Even, J3 Conn_01x06, Q1 NPN_2N3904_SOT23, SW1 Omron_B3F_SPST, SW2 Omron_B3F_SPST, SW3 Omron_B3F_SPST, SW4 Omron_B3F_SPST, U1 ATmega328-PU, U2 MAX7219, U3 DS1307_DIP-8, U4 L7805, Y1 Crystal_16MHz, Y2 Crystal_32768Hz

Commit message: Final Gerber
Git commit for final Gerber Out. I forgot to upload the Google Form for the initial Gerber but everything from the first one is in the previous Git commit.
Parts:
- added TP15: TestPoint, footprints:TestPoint_THTPad_D2.0mm_Drill1.0mm, F.Cu at (121.2, 81.0)
- added TP16: TestPoint, footprints:TestPoint_THTPad_D2.0mm_Drill1.0mm, F.Cu at (98.0, 140.0)
- added TP17: TestPoint, footprints:TestPoint_THTPad_D2.0mm_Drill1.0mm, F.Cu at (103.0, 140.0)
- added TP18: TestPoint, footprints:TestPoint_THTPad_D2.0mm_Drill1.0mm, F.Cu at (108.0, 140.0)
- added TP19: TestPoint, footprints:TestPoint_THTPad_D2.0mm_Drill1.0mm, F.Cu at (113.8, 87.5)
- added TP20: TestPoint, footprints:TestPoint_THTPad_D2.0mm_Drill1.0mm, F.Cu at (107.2, 97.2)
- J1: value VAL** -> PJ-102AH
- moved J1 5.12 mm to (202.6, 134.7), turned to 180 degrees
Routing:
- net Net-(C7-Pad1): track 22.6 -> 59.8 mm
- net SCL: track 52.0 -> 74.5 mm, vias 2 -> 5
- net SDA: track 45.1 -> 54.0 mm
- net DIS_DATA: track 140.2 -> 147.9 mm
- net LED_SCK: track 55.0 -> 62.5 mm
- net DIS_CLK: track 99.0 -> 104.2 mm
- net DIS_LOAD: track 117.6 -> 121.8 mm

Commit message: Gerber Out Revisions 1
Parts:
- removed TP2, TP3, TP4, TP6, TP7, TP9: TestPoint, footprints:TestPoint_THTPad_D2.0mm_Drill1.0mm
- moved TP12 20.8 mm to (126.8, 102.5)
- moved TP11 12.2 mm to (152.0, 102.8)
- moved R9 0.36 mm to (185.8, 101.8)
Connections:
- net LCD_1 renamed RS
- net LCD_2 renamed E
- net LCD_3 renamed D4
- net LCD_4 renamed D5
- net LCD_5 renamed D6
- net LCD_6 renamed D7
- TP11 pad 1: GND -> Net-(DS1-Pad15)
- U1 pad 22: unconnected-(U1-Pad22) -> GND
Routing:
- net VCC: track 0.00 -> 40.1 mm, vias 0 -> 4
- net Net-(DS1-Pad15): track 4.11 -> 9.00 mm
- net Net-(C7-Pad1): track 59.8 -> 61.7 mm

Commit message: Final Gerber Out (with revisions)
Parts:
- J1: value PJ-102AH -> VAL**
- moved C6 1.57 mm to (209.0, 87.8)
- moved R12 1.47 mm to (209.1, 82.5)
- moved R11 1.38 mm to (209.0, 85.0)
Routing:
- net VCC: track 40.1 -> 9.95 mm, vias 4 -> 2
- net Net-(DS1-Pad3): track 111.6 -> 115.4 mm
- net RXD: track 133.5 -> 136.9 mm
- net TXD: track 141.7 -> 144.8 mm
- net RESET: track 150.6 -> 148.9 mm
- net /SER_TX: track 4.76 -> 3.43 mm
- net /SER_RX: track 4.76 -> 3.55 mm
- net /RTS: track 4.76 -> 3.56 mm
- net D4: track 45.3 -> 44.7 mm
